File: addon/kicad/mini_meow.kicad_pcb (KiCad board)
At the start: 2 copper layers, 0 parts

Commit message: updated kicad for new layout
Parts:
- added D1: LED, LEDs:LED_D5.0mm, F.Cu at (130.0, 118.1)
- added D2: LED, LEDs:LED_D5.0mm, F.Cu at (114.8, 118.1)
- added R1: 65, Resistors_THT:R_Axial_DIN0204_L3.6mm_D1.6mm_P7.62mm_Horizontal, F.Cu at (123.2, 126.5)
- added R2: 65, Resistors_THT:R_Axial_DIN0204_L3.6mm_D1.6mm_P7.62mm_Horizontal, F.Cu at (118.1, 126.2)
- added U1: sa_connector, Pin_Headers:Pin_Header_Straight_2x02_Pitch2.54mm, F.Cu at (133.9, 145.0)
