File: addon/kicad/mini_meow.sch (KiCad schematic (older format))
At the start: 4 parts

Commit message: added ground
Connections:
- net GND: now reaches D?.1 (K), D?.1 (K), U?.2 (GND)
Changed lines of the file:
@@
 	5850 4800 5850 4350
 Connection ~ 4650 4550
+$Comp
+L GND #PWR?
+U 1 1 5B47CD76
+P 5300 4950
+F 0 "#PWR?" H 5300 4700 50  0001 C CNN
+F 1 "GND" H 5300 4800 50  0000 C CNN
+F 2 "" H 5300 4950 50  0001 C CNN
+F 3 "" H 5300 4950 50  0001 C CNN
+	1    5300 4950
+	1    0    0    -1
+$EndComp
+Wire Wire Line
+	5300 4950 5300 4800
+Connection ~ 5300 4800
 $EndSCHEMATC

Commit message: added net list, updated schematic, layout
Parts:
- added R2: 51, symbol R
- R1: renamed from R?; value R -> 51
- gave numbers to parts that had none: 3
Connections:
- net GND: now also R2.2
- net at D1.2 (A), R1.1: no longer D2.2 (A)
- new net: D2.2 (A), R2.1
Changed lines of the file:
@@
 $EndDescr
 $Comp
-L LED_ALT D?
+L LED_ALT D1
 U 1 1 5B453E32
 P 5050 4050
-F 0 "D?" H 5050 4150 50  0000 C CNN
+F 0 "D1" H 5050 4150 50  0000 C CNN
 F 1 "LED" H 5050 3950 50  0000 C CNN
 F 2 "" H 5050 4050 50  0001 C CNN
@@
 $EndComp
 $Comp
-L LED_ALT D?
+L LED_ALT D2
 U 1 1 5B453E73
 P 5050 4550
-F 0 "D?" H 5050 4650 50  0000 C CNN
+F 0 "D2" H 5050 4650 50  0000 C CNN
 F 1 "LED" H 5050 4450 50  0000 C CNN
 F 2 "" H 5050 4550 50  0001 C CNN
@@
 $EndComp
 $Comp
-L sa_connector U?
+L sa_connector U1
 U 1 1 5B454775
 P 6250 4350
-F 0 "U?" H 6450 4175 60  0000 C CNN
+F 0 "U1" H 6450 4175 60  0000 C CNN
 F 1 "sa_connector" H 6275 4600 60  0000 C CNN
 F 2 "" H 6275 4375 60  0001 C CNN
@@
 $EndComp
 $Comp
-L R R?
+L R R1
 U 1 1 5B45481B
 P 5500 4250
-F 0 "R?" V 5580 4250 50  0000 C CNN
-F 1 "R" V 5500 4250 50  0000 C CNN
+F 0 "R1" V 5580 4250 50  0000 C CNN
+F 1 "51" V 5500 4250 50  0000 C CNN
 F 2 "" V 5430 4250 50  0001 C CNN
 F 3 "" H 5500 4250 50  0001 C CNN
@@
 	0    -1   -1   0
 $EndComp
+$Comp
+L GND #PWR01
+U 1 1 5B47CD76
+P 5300 4950
+F 0 "#PWR01" H 5300 4700 50  0001 C CNN
+F 1 "GND" H 5300 4800 50  0000 C CNN
+F 2 "" H 5300 4950 50  0001 C CNN
+F 3 "" H 5300 4950 50  0001 C CNN
+	1    5300 4950
+	1    0    0    -1
+$EndComp
+$Comp
+L R R2
+U 1 1 5B48B2F9
+P 5500 4450
+F 0 "R2" V 5580 4450 50  0000 C CNN
+F 1 "51" V 5500 4450 50  0000 C CNN
+F 2 "" V 5430 4450 50  0001 C CNN
+F 3 "" H 5500 4450 50  0001 C CNN
+	1    5500 4450
+	0    -1   -1   0
+$EndComp
 Wire Wire Line
 	5850 4250 5650 4250
 Wire Wire Line
-	5200 4050 5200 4550
+	5200 4050 5200 4250
 Wire Wire Line
 	5200 4250 5350 4250
-Connection ~ 5200 4250
 Wire Wire Line
 	4900 4050 4650 4050
@@
 	5850 4800 5850 4350
 Connection ~ 4650 4550
-$Comp
-L GND #PWR?
-U 1 1 5B47CD76
-P 5300 4950
-F 0 "#PWR?" H 5300 4700 50  0001 C CNN
-F 1 "GND" H 5300 4800 50  0000 C CNN
-F 2 "" H 5300 4950 50  0001 C CNN
-F 3 "" H 5300 4950 50  0001 C CNN
-	1    5300 4950
-	1    0    0    -1
-$EndComp
 Wire Wire Line
 	5300 4950 5300 4800
 Connection ~ 5300 4800
+Wire Wire Line
+	5650 4450 5650 4350
+Wire Wire Line
+	5650 4350 5850 4350
+Wire Wire Line
+	5350 4450 5250 4450
+Wire Wire Line
+	5250 4450 5250 4550
+Wire Wire Line
+	5250 4550 5200 4550
 $EndSCHEMATC

Commit message: moved back from 2 resistors to 1
Parts:
- removed R2: 51, symbol R
Connections:
- net at D1.2 (A), R1.1: now also D2.2 (A)
Changed lines of the file:
@@
 	1    0    0    -1
-$EndComp
-$Comp
-L R R2
-U 1 1 5B48B2F9
-P 5500 4450
-F 0 "R2" V 5580 4450 50  0000 C CNN
-F 1 "51" V 5500 4450 50  0000 C CNN
-F 2 "" V 5430 4450 50  0001 C CNN
-F 3 "" H 5500 4450 50  0001 C CNN
-	1    5500 4450
-	0    -1   -1   0
 $EndComp
 Wire Wire Line
 	5850 4250 5650 4250
 Wire Wire Line
-	5200 4050 5200 4250
-Wire Wire Line
-	5200 4250 5350 4250
+	5250 4050 5250 4550
 Wire Wire Line
 	4900 4050 4650 4050
@@
 Connection ~ 5300 4800
 Wire Wire Line
-	5650 4450 5650 4350
+	5250 4550 5200 4550
 Wire Wire Line
-	5650 4350 5850 4350
+	5250 4050 5200 4050
 Wire Wire Line
-	5350 4450 5250 4450
-Wire Wire Line
-	5250 4450 5250 4550
-Wire Wire Line
-	5250 4550 5200 4550
+	5350 4250 5250 4250
+Connection ~ 5250 4250
 $EndSCHEMATC

Commit message: updated kicad for new layout
Parts:
- added R2: 65, Resistors_THT:R_Axial_DIN0204_L3.6mm_D1.6mm_P7.62mm_Horizontal, symbol R
- D1, D2: footprint (none) -> LEDs:LED_D5.0mm
- R1: value 51 -> 65; footprint (none) -> Resistors_THT:R_Axial_DIN0207_L6.3mm_D2.5mm_P7.62mm_Horizontal
- U1: footprint (none) -> Pin_Headers:Pin_Header_Straight_2x02_Pitch2.54mm
Connections:
- net at D1.2 (A), R1.1: no longer D2.2 (A)
- net +3V3: now reaches R1.2, U1.1 (VCC)
- net +3V3: now also R2.2
- new net: D2.2 (A), R2.1
Other:
- moved on the sheet: D1, D2, R1
Changed lines of the file:
@@
 L LED_ALT D1
 U 1 1 5B453E32
-P 5050 4050
-F 0 "D1" H 5050 4150 50  0000 C CNN
-F 1 "LED" H 5050 3950 50  0000 C CNN
-F 2 "" H 5050 4050 50  0001 C CNN
-F 3 "" H 5050 4050 50  0001 C CNN
-	1    5050 4050
+P 4950 4050
+F 0 "D1" H 4950 4150 50  0000 C CNN
+F 1 "LED" H 4950 3950 50  0000 C CNN
+F 2 "LEDs:LED_D5.0mm" H 4950 4050 50  0001 C CNN
+F 3 "" H 4950 4050 50  0001 C CNN
+	1    4950 4050
 	1    0    0    -1
 $EndComp
@@
 L LED_ALT D2
 U 1 1 5B453E73
-P 5050 4550
-F 0 "D2" H 5050 4650 50  0000 C CNN
-F 1 "LED" H 5050 4450 50  0000 C CNN
-F 2 "" H 5050 4550 50  0001 C CNN
-F 3 "" H 5050 4550 50  0001 C CNN
-	1    5050 4550
+P 4950 4550
+F 0 "D2" H 4950 4650 50  0000 C CNN
+F 1 "LED" H 4950 4450 50  0000 C CNN
+F 2 "LEDs:LED_D5.0mm" H 4950 4550 50  0001 C CNN
+F 3 "" H 4950 4550 50  0001 C CNN
+	1    4950 4550
 	1    0    0    -1
 $EndComp
@@
 F 0 "U1" H 6450 4175 60  0000 C CNN
 F 1 "sa_connector" H 6275 4600 60  0000 C CNN
-F 2 "" H 6275 4375 60  0001 C CNN
+F 2 "Pin_Headers:Pin_Header_Straight_2x02_Pitch2.54mm" H 6275 4375 60  0001 C CNN
 F 3 "" H 6275 4375 60  0001 C CNN
 	1    6250 4350
@@
 L R R1
 U 1 1 5B45481B
-P 5500 4250
-F 0 "R1" V 5580 4250 50  0000 C CNN
-F 1 "51" V 5500 4250 50  0000 C CNN
-F 2 "" V 5430 4250 50  0001 C CNN
-F 3 "" H 5500 4250 50  0001 C CNN
-	1    5500 4250
+P 5400 4250
+F 0 "R1" V 5480 4250 50  0000 C CNN
+F 1 "65" V 5400 4250 50  0000 C CNN
+F 2 "Resistors_THT:R_Axial_DIN0207_L6.3mm_D2.5mm_P7.62mm_Horizontal" V 5330 4250 50  0001 C CNN
+F 3 "" H 5400 4250 50  0001 C CNN
+	1    5400 4250
 	0    -1   -1   0
 $EndComp
@@
 L GND #PWR01
 U 1 1 5B47CD76
-P 5300 4950
-F 0 "#PWR01" H 5300 4700 50  0001 C CNN
-F 1 "GND" H 5300 4800 50  0000 C CNN
-F 2 "" H 5300 4950 50  0001 C CNN
-F 3 "" H 5300 4950 50  0001 C CNN
-	1    5300 4950
+P 5200 4950
+F 0 "#PWR01" H 5200 4700 50  0001 C CNN
+F 1 "GND" H 5200 4800 50  0000 C CNN
+F 2 "" H 5200 4950 50  0001 C CNN
+F 3 "" H 5200 4950 50  0001 C CNN
+	1    5200 4950
 	1    0    0    -1
 $EndComp
+$Comp
+L +3.3V #PWR02
+U 1 1 5B503505
+P 5850 4050
+F 0 "#PWR02" H 5850 3900 50  0001 C CNN
+F 1 "+3.3V" H 5850 4190 50  0000 C CNN
+F 2 "" H 5850 4050 50  0001 C CNN
+F 3 "" H 5850 4050 50  0001 C CNN
+	1    5850 4050
+	1    0    0    -1
+$EndComp
+$Comp
+L R R2
+U 1 1 5B5046EC
+P 5400 4450
+F 0 "R2" V 5480 4450 50  0000 C CNN
+F 1 "65" V 5400 4450 50  0000 C CNN
+F 2 "Resistors_THT:R_Axial_DIN0204_L3.6mm_D1.6mm_P7.62mm_Horizontal" V 5330 4450 50  0001 C CNN
+F 3 "" H 5400 4450 50  0001 C CNN
+	1    5400 4450
+	0    -1   -1   0
+$EndComp
 Wire Wire Line
-	5850 4250 5650 4250
+	5150 4050 5150 4250
 Wire Wire Line
-	5250 4050 5250 4550
+	4800 4050 4550 4050
 Wire Wire Line
-	4900 4050 4650 4050
+	4550 4050 4550 4800
 Wire Wire Line
-	4650 4050 4650 4800
+	4550 4550 4800 4550
 Wire Wire Line
-	4650 4550 4900 4550
-Wire Wire Line
-	4650 4800 5850 4800
+	4550 4800 5850 4800
 Wire Wire Line
 	5850 4800 5850 4350
-Connection ~ 4650 4550
+Connection ~ 4550 4550
 Wire Wire Line
-	5300 4950 5300 4800
-Connection ~ 5300 4800
+	5200 4950 5200 4800
+Connection ~ 5200 4800
 Wire Wire Line
-	5250 4550 5200 4550
+	5150 4050 5100 4050
 Wire Wire Line
-	5250 4050 5200 4050
+	5150 4250 5250 4250
 Wire Wire Line
-	5350 4250 5250 4250
-Connection ~ 5250 4250
+	5850 4050 5850 4250
+Wire Wire Line
+	5100 4550 5150 4550
+Wire Wire Line
+	5150 4550 5150 4450
+Wire Wire Line
+	5150 4450 5250 4450
+Wire Wire Line
+	5850 4250 5550 4250
+Wire Wire Line
+	5550 4450 5650 4450
+Wire Wire Line
+	5650 4450 5650 4250
+Connection ~ 5650 4250
 $EndSCHEMATC

Commit message: pcb update, added working art files
Parts:
- R1: footprint Resistors_THT:R_Axial_DIN0207_L6.3mm_D2.5mm_P7.62mm_Horizontal -> Resistors_THT:R_Axial_DIN0204_L3.6mm_D1.6mm_P7.62mm_Horizontal
Changed lines of the file:
@@
 F 0 "R1" V 5480 4250 50  0000 C CNN
 F 1 "65" V 5400 4250 50  0000 C CNN
-F 2 "Resistors_THT:R_Axial_DIN0207_L6.3mm_D2.5mm_P7.62mm_Horizontal" V 5330 4250 50  0001 C CNN
+F 2 "Resistors_THT:R_Axial_DIN0204_L3.6mm_D1.6mm_P7.62mm_Horizontal" V 5330 4250 50  0001 C CNN
 F 3 "" H 5400 4250 50  0001 C CNN
 	1    5400 4250

Commit message: updated mask for copper
Parts:
- R1, R2: value 65 -> 68
Changed lines of the file:
@@
 P 5400 4250
 F 0 "R1" V 5480 4250 50  0000 C CNN
-F 1 "65" V 5400 4250 50  0000 C CNN
+F 1 "68" V 5400 4250 50  0000 C CNN
 F 2 "Resistors_THT:R_Axial_DIN0204_L3.6mm_D1.6mm_P7.62mm_Horizontal" V 5330 4250 50  0001 C CNN
 F 3 "" H 5400 4250 50  0001 C CNN
@@
 P 5400 4450
 F 0 "R2" V 5480 4450 50  0000 C CNN
-F 1 "65" V 5400 4450 50  0000 C CNN
+F 1 "68" V 5400 4450 50  0000 C CNN
 F 2 "Resistors_THT:R_Axial_DIN0204_L3.6mm_D1.6mm_P7.62mm_Horizontal" V 5330 4450 50  0001 C CNN
 F 3 "" H 5400 4450 50  0001 C CNN
