File: pcb/eagle/dc26_maneki-neko_badge_VERSION2.brd (EAGLE design)
At the start: 75.8 x 126.7 mm, 53 parts, among them SW1 PTS645SM43SMTR92, T1 RK7002BMT116, U1 STM32F030C8T, U2 PAM2301CAAB330, U3 NPTC042KFMS-RC

Commit message: pcb v2 routed, bom edited, gerbers rendered - quote out to pcba house and dfm check to freedfm
Parts:
- moved R30 113.3 mm to (27.5, 102.4), flipped to the bottom, turned to 270 degrees
- moved S2 91.1 mm to (55.7, 68.2), flipped to the bottom, turned to 90 degrees
- moved R29 1.61 mm to (32.7, 102.0)
- moved R28 1.61 mm to (30.5, 102.0)
- renumbered U$2 to H4
Connections:
- removed net ESP-!FAULT: U1.33
- removed net ESP-EN: U1.30
- removed net LEFT-EYE-!FAULT: U1.31
- removed net RIGHT-EYE-!FAULT: U1.32
Routing:
- net ESP-EN: track 65.6 -> 0.00 mm, vias 2 -> 0
- net RIGHT-EYE-!FAULT: track 65.5 -> 0.00 mm, vias 2 -> 0
- net ESP-!FAULT: track 50.7 -> 0.00 mm, vias 2 -> 0
- net LEFT-EYE-!FAULT: track 44.0 -> 0.00 mm, vias 2 -> 0
- net ESP-VCC: track 3.54 -> 32.2 mm, vias 0 -> 2
- net 3V3: track 68.5 -> 84.3 mm, vias 14 -> 15
- net V2_CHECK: track 0.00 -> 10.6 mm
- net N$5: track 0.00 -> 2.03 mm
- net BOOT0: track 14.7 -> 16.3 mm
- net GND: vias 20 -> 18
